File: mars_rover_navigation_system.kicad_sch (KiCad schematic)
At the start: 7 parts, among them U1 ESP32-WROOM-32, U2 AM2302, U3 BQ24090DGQ

Commit message: added title
Other:
- title: (none) -> MRNOS
Changed lines of the file:
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@@
 	(generator_version "8.0")
 	(paper "A5")
+	(title_block
+		(title "MRNOS")
+		(date "2025-02-10")
+		(rev "v.1")
+	)
 	(junction
 		(at 83.82 44.45)
